File: sensor-node.kicad_pcb (KiCad board)
At the start: 2 copper layers, 63.5 x 63.5 mm, 51 parts, among them J1 DIGITAL_IN, J10 I2C, J11 ANALOG_IN, J12 +5, J2 DIGITAL_OUT, J3 +24, J4 GND, J5 CANH_TERM, J6 CANL_TERM, J7 RJ45_A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

Commit message: Osh Park label Done
Parts:
- J12: value +5 -> +5V
- J3: value +24 -> +24V
Routing:
- net GND: track 483.5 -> 480.5 mm, vias 15 -> 13
- net (no net): track 0.00 -> 2.96 mm, vias 0 -> 2
Other:
- rule pad_to_mask_clearance: 0.2 -> 0.0762
- board text added: "Analog In"
- board text added: "Digital In"
- board text added: "Digital Out"
- board text added: "I2C"
Changed lines of the file:
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@@
     (area 50.724999 25.324999 114.4874 88.975001)
     (thickness 1.6)
-    (drawings 4)
+    (drawings 8)
     (tracks 584)
     (zones 0)
@@
   )
   (setup
-    (last_trace_width 0.381)
+    (last_trace_width 0.1524)
     (user_trace_width 0.254)
     (user_trace_width 0.381)
@@
     (pad_size 1.524 1.524)
     (pad_drill 0.762)
-    (pad_to_mask_clearance 0.2)
+    (pad_to_mask_clearance 0.0762)
     (aux_axis_origin 0 0)
     (grid_origin 85.725 81.2)
@@
     (tags "SMD SMT crystal hand-soldering")
     (attr smd)
-    (fp_text reference Y1 (at 5.0635 3.683 270) (layer F.SilkS)
+    (fp_text reference Y1 (at 8.5598 3.683 270) (layer F.SilkS)
       (effects (font (size 1 1) (thickness 0.15)))
     )
@@
     (at 55.88 30.48)
     (tags RJ45)
-    (fp_text reference J7 (at -0.5715 15.795) (layer F.SilkS)
+    (fp_text reference J7 (at -3.7592 15.4267) (layer F.SilkS)
       (effects (font (size 1 1) (thickness 0.15)))
     )
@@
     (at 81.28 40.814 180)
     (tags RJ45)
-    (fp_text reference J9 (at -6.35 13.1445 180) (layer F.SilkS)
+    (fp_text reference J9 (at -4.4831 13.4239 180) (layer F.SilkS)
       (effects (font (size 1 1) (thickness 0.15)))
     )
@@
     (tags "CMS SOT")
     (attr smd)
-    (fp_text reference U1 (at 0 -4.5 270) (layer F.SilkS)
+    (fp_text reference U1 (at -5.2451 0.127 360) (layer F.SilkS)
       (effects (font (size 1 1) (thickness 0.15)))
     )
@@
     (tags "capacitor 0805")
     (attr smd)
-    (fp_text reference C1 (at 0 -1.75 270) (layer F.SilkS)
+    (fp_text reference C1 (at -3.429 -0.0762 270) (layer F.SilkS)
       (effects (font (size 1 1) (thickness 0.15)))
     )
@@
     (tags "capacitor 1210")
     (attr smd)
-    (fp_text reference C2 (at 0 -2.25 90) (layer F.SilkS)
+    (fp_text reference C2 (at -4.2164 0.1905 90) (layer F.SilkS)
       (effects (font (size 1 1) (thickness 0.15)))
     )
@@
     (tags "capacitor 0805")
     (attr smd)
-    (fp_text reference C5 (at 3.382 0.889 270) (layer F.SilkS)
+    (fp_text reference C5 (at 1.2573 -1.9558 270) (layer F.SilkS)
       (effects (font (size 1 1) (thickness 0.15)))
     )
@@
     (tags "capacitor 0805")
     (attr smd)
-    (fp_text reference C6 (at -1.063 -1.397 270) (layer F.SilkS)
+    (fp_text reference C6 (at 3.4671 -0.8509 270) (layer F.SilkS)
       (effects (font (size 1 1) (thickness 0.15)))
     )
@@
     (tags "capacitor 0805")
     (attr smd)
-    (fp_text reference C8 (at 0 -1.75 90) (layer F.SilkS)
+    (fp_text reference C8 (at 2.8448 0.0635 180) (layer F.SilkS)
       (effects (font (size 1 1) (thickness 0.15)))
     )
@@
   (module ab2_connector:AB2_0.25_QD_TAB (layer F.Cu)
     (at 106.68 30.48 180)
-    (fp_text reference J3 (at -5.1435 1.2865 180) (layer F.SilkS)
+    (fp_text reference J3 (at -0.0254 -1.444 180) (layer F.SilkS)
       (effects (font (size 0.8128 0.8128) (thickness 0.0762)))
     )
-    (fp_text value +24 (at -5.715 0.08 180) (layer F.SilkS)
-      (effects (font (size 0.8128 0.8128) (thickness 0.0762)))
+    (fp_text value +24V (at -4.3053 2.62 180) (layer F.SilkS)
+      (effects (font (size 1.143 1.143) (thickness 0.0762)))
     )
     (fp_line (start 1.8415 -0.381) (end 1.7145 -0.254) (layer F.SilkS) (width 0.0762))
@@
   (module ab2_connector:AB2_0.25_QD_TAB (layer F.Cu)
     (at 106.68 40.64 180)
-    (fp_text reference J4 (at -5.08 -1.317 180) (layer F.SilkS)
+    (fp_text reference J4 (at -0.0635 -1.5837 180) (layer F.SilkS)
       (effects (font (size 0.8128 0.8128) (thickness 0.0762)))
     )
-    (fp_text value GND (at -5.5245 0.334 180) (layer F.SilkS)
-      (effects (font (size 0.8128 0.8128) (thickness 0.0762)))
+    (fp_text value GND (at -4.8514 2.0485 180) (layer F.SilkS)
+      (effects (font (size 1.143 1.143) (thickness 0.0762)))
     )
     (fp_line (start 1.8415 -0.381) (end 1.7145 -0.254) (layer F.SilkS) (width 0.0762))
@@
     (descr "Through hole straight pin header, 1x02, 2.54mm pitch, single row")
     (tags "Through hole pin header THT 1x02 2.54mm single row")
-    (fp_text reference J5 (at -5.461 2.7305) (layer F.SilkS)
+    (fp_text reference J5 (at -0.0635 5.1562) (layer F.SilkS)
       (effects (font (size 1 1) (thickness 0.15)))
     )
@@
     (descr "Through hole straight pin header, 2x05, 1.27mm pitch, double rows")
     (tags "Through hole pin header THT 2x05 1.27mm double row")
-    (fp_text reference J8 (at 0.635 -1.695) (layer F.SilkS)
+    (fp_text reference J8 (at 0.7493 -2.6162) (layer F.SilkS)
       (effects (font (size 1 1) (thickness 0.15)))
     )
@@
   (module ab2_connector:AB2_0.25_QD_TAB (layer F.Cu)
     (at 106.68 35.56 180)
-    (fp_text reference J12 (at -5.715 1.35 180) (layer F.SilkS)
+    (fp_text reference J12 (at 0.1016 -1.4567 180) (layer F.SilkS)
       (effects (font (size 0.8128 0.8128) (thickness 0.0762)))
     )
-    (fp_text value +5 (at -5.715 0.08 180) (layer F.SilkS)
-      (effects (font (size 0.8128 0.8128) (thickness 0.0762)))
+    (fp_text value +5V (at -4.699 2.112 180) (layer F.SilkS)
+      (effects (font (size 1.143 1.143) (thickness 0.0762)))
     )
     (fp_line (start 1.8415 -0.381) (end 1.7145 -0.254) (layer F.SilkS) (width 0.0762))
@@
     (tags "resistor 0805")
     (attr smd)
-    (fp_text reference R12 (at 0 -1.7 180) (layer F.SilkS)
+    (fp_text reference R12 (at -0.2794 1.5875 180) (layer F.SilkS)
       (effects (font (size 1 1) (thickness 0.15)))
     )
@@
     (tags "resistor 0805")
     (attr smd)
-    (fp_text reference R13 (at 0 -1.7 180) (layer F.SilkS)
+    (fp_text reference R13 (at -5.1816 0.2413 180) (layer F.SilkS)
       (effects (font (size 1 1) (thickness 0.15)))
     )
@@
     (tags "SOP 1.27")
     (attr smd)
-    (fp_text reference U2 (at -0.047 2.921 90) (layer F.SilkS)
+    (fp_text reference U2 (at -0.2248 2.7686 90) (layer F.SilkS)
       (effects (font (size 1 1) (thickness 0.15)))
     )
@@
     (tags "QFP 0.8")
     (attr smd)
-    (fp_text reference U4 (at 0 -5.85) (layer F.SilkS)
+    (fp_text reference U4 (at 1.8542 -6.3284) (layer F.SilkS)
       (effects (font (size 1 1) (thickness 0.15)))
     )
@@
     (tags "resistor 0805")
     (attr smd)
-    (fp_text reference R9 (at 0 -1.7) (layer F.SilkS)
+    (fp_text reference R9 (at -1.3208 1.6764) (layer F.SilkS)
       (effects (font (size 1 1) (thickness 0.15)))
     )
@@
     (tags "resistor 0805")
     (attr smd)
-    (fp_text reference R10 (at 0 -1.7) (layer F.SilkS)
+    (fp_text reference R10 (at -2.667 1.5494) (layer F.SilkS)
       (effects (font (size 1 1) (thickness 0.15)))
     )
@@
     (tags "resistor 0805")
     (attr smd)
-    (fp_text reference R16 (at 0 -1.7) (layer F.SilkS)
+    (fp_text reference R16 (at 2.7432 1.6129) (layer F.SilkS)
       (effects (font (size 1 1) (thickness 0.15)))
     )
@@
     )
   )
+  (gr_text "Digital\nIn" (at 56.134 49.8945) (layer F.SilkS)
+    (effects (font (size 1.5 1.5) (thickness 0.3)))
+  )
+  (gr_text "Analog \nIn" (at 56.6166 86.3308) (layer F.SilkS)
+    (effects (font (size 1.5 1.5) (thickness 0.3)))
+  )
+  (gr_text "Digital\nOut" (at 106.7054 86.3308) (layer F.SilkS)
+    (effects (font (size 1.5 1.5) (thickness 0.3)))
+  )
+  (gr_text I2C (at 106.6165 66.1632) (layer F.SilkS)
+    (effects (font (size 1.5 1.5) (thickness 0.3)))
+  )
   (gr_line (start 50.8 88.9) (end 50.8 25.4) (angle 90) (layer Edge.Cuts) (width 0.15))
   (gr_line (start 114.3 88.9) (end 50.8 88.9) (angle 90) (layer Edge.Cuts) (width 0.15))
   (gr_line (start 114.3 25.4) (end 114.3 88.9) (angle 90) (layer Edge.Cuts) (width 0.15))
   (gr_line (start 50.8 25.4) (end 114.3 25.4) (angle 90) (layer Edge.Cuts) (width 0.15))
+  (via (at 110.5789 67.1411) (size 0.6858) (drill 0.3302) (layers F.Cu B.Cu) (net 0))
+  (segment (start 110.5789 67.1411) (end 112.0902 65.6298) (width 0.381) (layer B.Cu) (net 0))
+  (segment (start 112.0902 65.6298) (end 112.0902 64.8043) (width 0.381) (layer B.Cu) (net 0))
+  (via (at 112.0902 64.8043) (size 0.6858) (drill 0.3302) (layers F.Cu B.Cu) (net 0))
   (segment (start 55.88 30.48) (end 54.3014 30.48) (width 0.254) (layer B.Cu) (net 1))
   (segment (start 70.9358 80.076) (end 69.934 80.076) (width 0.254) (layer F.Cu) (net 1))
@@
   (segment (start 55.88 30.48) (end 55.88 29.21) (width 0.381) (layer F.Cu) (net 1))
   (segment (start 55.88 29.21) (end 57.15 27.94) (width 0.381) (layer F.Cu) (net 1))
-  (via (at 110.5789 67.1411) (size 0.6858) (drill 0.3302) (layers F.Cu B.Cu) (net 2))
-  (segment (start 110.5789 67.1411) (end 112.0902 65.6298) (width 0.381) (layer B.Cu) (net 2))
-  (segment (start 112.0902 65.6298) (end 112.0902 64.8043) (width 0.381) (layer B.Cu) (net 2))
-  (via (at 112.0902 64.8043) (size 0.6858) (drill 0.3302) (layers F.Cu B.Cu) (net 2))
   (segment (start 109.22 40.64) (end 111.713 40.64) (width 0.381) (layer B.Cu) (net 2))
   (segment (start 111.713 40.64) (end 113.2967 39.0563) (width 0.381) (layer B.Cu) (net 2))
